Commit message: With Gazebo only break

File: urdf/robot_xacro.xacro (robot description, xacro)
@@ -8,4 +8,11 @@
      For more information, please see http://wiki.ros.org/sw_urdf_exporter -->
 <robot name="Robot1" xmlns:xacro="http://ros.org/wiki/xacro">
+<xacro:include filename="$(find urdf_test)/gazebo/robot.gazebo" />
+  <link name="dummy">
+    </link>
+  <joint name="dummy_joint" type="fixed">
+    <parent link="dummy"/>
+    <child link="base_link"/>
+  </joint>
   <link name="base_link">
     <inertial>

Commit message: Break branch

File: urdf/robot_xacro.xacro (robot description, xacro)
@@ -1,3 +1,2 @@
-<?xml version="1.0" ?>
 <!-- =================================================================================== -->
 <!-- |    This document was autogenerated by xacro from robot.urdf                     | -->
@@ -8,11 +7,11 @@
      For more information, please see http://wiki.ros.org/sw_urdf_exporter -->
 <robot name="Robot1" xmlns:xacro="http://ros.org/wiki/xacro">
-<xacro:include filename="$(find urdf_test)/gazebo/robot.gazebo" />
+  <xacro:include filename="$(find urdf_test)/gazebo/robot.gazebo" />
   <link name="dummy">
     </link>
-  <joint name="dummy_joint" type="fixed">
+    <joint name="dummy_joint" type="fixed">
     <parent link="dummy"/>
     <child link="base_link"/>
-  </joint>
+    </joint>
   <link name="base_link">
     <inertial>
